File: SuperDoppler2000.kicad_sch (KiCad schematic)
At the start: 5 parts, among them U1 TPS7A0533PDBZ

Commit message: Add files via upload
Other:
- note added: "Vin ?? 4.5 or 6"
- note removed: "Vin ??"
Changed lines of the file:
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@@
 	)
 	(rectangle
-		(start 26.67 27.94)
-		(end 80.01 68.58)
+		(start 26.67 30.48)
+		(end 80.01 71.12)
 		(stroke
 			(width 0)
@@
 		)
 	)
-	(text "Vin ??\n"
+	(text "Vin ?? 4.5 or 6 \n"
 		(exclude_from_sim no)
 		(at 166.624 33.274 0)
